File: PMW3360_PCB/PMW3360_PCB.kicad_pcb (KiCad board)
At the start: 2 copper layers, 34.3 x 45.7 mm, 26 parts, among them J1 Conn_02x04_Odd_Even, J2 Conn_01x08_MountingPin, U1 PMW3360DM-T2QU, U2 AP7361-18ER-13, U3 TXS0108E

Commit message: Update
Parts:
- removed C5, C6: 1uF, Capacitor_SMD:C_0603_1608Metric_Pad1.08x0.95mm_HandSolder
- removed J2: Conn_01x08_MountingPin, PMW3360_PCB:Molex 52271-0879 FFC FPC 8 Pin 1.0mm Pitch
- removed the REF** at (139.7, 85.9)
- removed the REF** at (139.7, 125.0)
- removed the REF** at (167.6, 85.9)
- removed the REF** at (167.6, 125.0)
- removed SB1: SolderJumper_3_Bridged12, Jumper:SolderJumper-3_P2.0mm_Open_TrianglePad1.0x1.5mm_NumberLabels
- removed SB2, SB3, SB4, SB5, SB6, SB7, SB8: SolderJumper_2_Open, Jumper:SolderJumper-2_P1.3mm_Open_TrianglePad1.0x1.5mm
- removed U3: TXS0108E, PMW3360_PCB:TSSOP-20
- added JP1: SolderJumper_3_Open, Jumper:SolderJumper-3_P1.3mm_Open_Pad1.0x1.5mm_NumberLabels, F.Cu at (237.4, 136.8)
- added R4: 56.2k, Resistor_SMD:R_0603_1608Metric_Pad0.98x0.95mm_HandSolder, F.Cu at (230.6, 155.0)
- added REF**: MountingHole_3.2mm_M3_DIN965_Pad, MountingHole:MountingHole_3.2mm_M3_DIN965_Pad, F.Cu at (236.6, 153.2)
- added REF**: MountingHole_3.2mm_M3_DIN965_Pad, MountingHole:MountingHole_3.2mm_M3_DIN965_Pad, F.Cu at (217.3, 153.2)
- added REF**: MountingHole_3.2mm_M3_DIN965_Pad, MountingHole:MountingHole_3.2mm_M3_DIN965_Pad, F.Cu at (236.6, 125.1)
- added REF**: MountingHole_3.2mm_M3_DIN965_Pad, MountingHole:MountingHole_3.2mm_M3_DIN965_Pad, F.Cu at (217.3, 125.1)
- added TP1: VDDIO TestPoint, TestPoint:TestPoint_Pad_D1.5mm, F.Cu at (229.5, 125.1)
- added TP2: VDD TestPoint, TestPoint:TestPoint_Pad_D1.5mm, F.Cu at (226.2, 125.1)
- added TP3: GND TestPoint, TestPoint:TestPoint_Pad_D1.5mm, F.Cu at (222.9, 125.1)
- J1: value Conn_02x04_Odd_Even -> Conn_01x08; footprint Connector_PinHeader_2.54mm:PinHeader_2x04_P2.54mm_Vertical -> Connector_PinHeader_2.54mm:PinHeader_1x08_P2.54mm_Vertical
- R3: value 10k -> 28k
- U2: value AP7361-18ER-13 -> TPS73601DBV; footprint Package_TO_SOT_SMD:SOT-223-3_TabPin2 -> Package_TO_SOT_SMD:SOT-23-5
- moved C4 104.9 mm to (228.1, 154.1), turned to -90 degrees
- moved C3 103.5 mm to (221.9, 154.1), turned to -90 degrees
- moved U2 99.4 mm to (225.0, 154.1)
- moved R3 97.4 mm to (230.6, 153.2), turned to 0 degrees
- moved C1 85.9 mm to (237.6, 142.7)
- moved C2 85.8 mm to (237.6, 146.1)
- moved R1 84.7 mm to (220.5, 143.4), turned to 90 degrees
- moved U1 84.2 mm to (233.8, 147.0)
- moved R2 79.0 mm to (220.5, 138.6), turned to 90 degrees
- moved J1 53.8 mm to (215.8, 130.2)
Connections:
- C3 pad 1: Net-(C3-Pad1) -> +3V3
- C4 pad 1: VDD -> +1V8
- J1 pad 1: /V_IN -> /MOTION
- J1 pad 2: /SCLK_O -> /SCLK
- J1 pad 3: /MOTION_O -> /MOSI
- J1 pad 4: /MOSI_O -> /MISO
- J1 pad 5: /RESET_O -> /CS
- J1 pad 6: /MISO_O -> /RESET
- J1 pad 7: GND -> +3V3
- J1 pad 8: /CS_O -> GND
- R1 pad 1: VDD -> +1V8
- R2 pad 1: VDD -> VCC
- R3 pad 1: Net-(R3-Pad1) -> +1V8
- R3 pad 2: GND -> Net-(R3-Pad2)
- U1 pad 4: VDD -> +1V8
- U1 pad 5: VDD -> VCC
- U2 pad 1: Net-(C3-Pad1) -> +3V3
- U2 pad 3: VDD -> +3V3
Routing:
- net VDD: track 109.8 -> 0.00 mm, vias 2 -> 0
- net GND: track 63.2 -> 145.8 mm, vias 13 -> 12
- net /MISO_O: track 75.6 -> 0.00 mm, vias 1 -> 0
- net +1V8: track 0.00 -> 71.0 mm
- net /MOSI_O: track 64.8 -> 0.00 mm, vias 1 -> 0
- net /V_IN: track 61.7 -> 0.00 mm, vias 2 -> 0
- net /SCLK_O: track 58.7 -> 0.00 mm, vias 1 -> 0
- net VCC: track 0.00 -> 56.7 mm
- net /CS: track 62.2 -> 7.30 mm
- net /MOTION_O: track 53.0 -> 0.00 mm, vias 1 -> 0
- net /CS_O: track 52.3 -> 0.00 mm
- net +3V3: track 0.00 -> 51.0 mm, vias 0 -> 2
- net /MISO: track 54.2 -> 7.74 mm, vias 1 -> 0
- net /RESET_O: track 45.9 -> 0.00 mm, vias 3 -> 0
- net /MOSI: track 49.8 -> 7.93 mm, vias 1 -> 0
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Other:
- board size 34.3 x 45.7 mm -> 26.4 x 35.2 mm
- board text added: "3V3"
- board text added: "JP1: 1-2 3: V_{IO}=3.3V 1 2-3: V_{IO}=1.8V"
- board text added: "Motion"
- board text added: "PMW3360 PCB Rev 2.0"
- board text added: "SI"
- board text added: "SO"
- board text added: "~{CS}"
- board text added: "~{RST}"
- board text removed: "1"
- board text removed: "2"
- board text removed: "7"
- board text removed: "8"
- board text removed: "Config1: V_IN=1.8~2.1V SB1[1-2 3],SB2[OFF],SB3~8[ON] Config2: V_IN=2.8~5.5V SB1[1 2-3],SB2[ON],SB3~8[OFF]"
- board text removed: "MISO"
- board text removed: "MOSI"
- board text removed: "MOTION"
- board text removed: "PMW3360 PCB Rev.1"
- board text removed: "V_IN"
- board text removed: "nCS"
- board text removed: "nRESET"
