File: PMW3360_PCB/PMW3360_PCB.kicad_sch (KiCad schematic)
At the start: 22 parts, among them J1 Conn_02x04_Odd_Even, J2 Conn_01x08_MountingPin, U1 PMW3360DM-T2QU, U2 AP7361-18ER-13, U3 TXS0108E-PWR

Commit message: Update
Parts:
- removed C5, C6: 1uF, Capacitor_SMD:C_0603_1608Metric_Pad1.08x0.95mm_HandSolder, symbol Device:C_Small
- removed J1: Conn_02x04_Odd_Even, Connector_PinHeader_2.54mm:PinHeader_2x04_P2.54mm_Vertical, symbol Connector_Generic:Conn_02x04_Odd_Even
- removed J2: Conn_01x08_MountingPin, PMW3360_PCB:Molex 52271-0879 FFC FPC 8 Pin 1.0mm Pitch, symbol Connector_Generic_MountingPin:Conn_01x08_MountingPin
- removed SB1: SolderJumper_3_Bridged12, Jumper:SolderJumper-3_P2.0mm_Open_TrianglePad1.0x1.5mm_NumberLabels, symbol Jumper:SolderJumper_3_Bridged12
- removed SB2, SB3, SB4, SB5, SB6, SB7, SB8: SolderJumper_2_Open, Jumper:SolderJumper-2_P1.3mm_Open_TrianglePad1.0x1.5mm, symbol Jumper:SolderJumper_2_Open
- removed U2: AP7361-18ER-13, Package_TO_SOT_SMD:SOT-223-3_TabPin2, symbol PMW3360_PCB:AP7361-18ER-13
- removed U3: TXS0108E-PWR, PMW3360_PCB:TSSOP-20, symbol PMW3360_PCB:TXS0108E-QPWRQ1
- added J1: Conn_01x08, Connector_PinHeader_2.54mm:PinHeader_1x08_P2.54mm_Vertical, symbol Connector_Generic:Conn_01x08
- added JP1: SolderJumper_3_Open, Jumper:SolderJumper-3_P1.3mm_Open_Pad1.0x1.5mm_NumberLabels, symbol Jumper:SolderJumper_3_Open
- added R4: 56.2k, Resistor_SMD:R_0603_1608Metric_Pad0.98x0.95mm_HandSolder, symbol Device:R
- added TP1: VDDIO TestPoint, TestPoint:TestPoint_Pad_D1.5mm, symbol Connector:TestPoint
- added TP2: VDD TestPoint, TestPoint:TestPoint_Pad_D1.5mm, symbol Connector:TestPoint
- added TP3: GND TestPoint, TestPoint:TestPoint_Pad_D1.5mm, symbol Connector:TestPoint
- added U2: TPS73601DBV, Package_TO_SOT_SMD:SOT-23-5, symbol Regulator_Linear:TPS73601DBV
- R3: value 10k -> 28k
Connections:
- net CS: now also J1.5 (Pin_5)
- net GND: now also J1.8 (Pin_8), R4.2, TP3.1, U2.2 (GND); no longer R3.2
- net MISO: now also J1.4 (Pin_4)
- net MOSI: now also J1.3 (Pin_3)
- net MOTION: now also J1.1 (Pin_1)
- net RESET: now also J1.6 (Pin_6)
- net SCLK: now also J1.2 (Pin_2)
- net +3V3: now reaches C3.1
- net +3V3: now also J1.7 (Pin_7), JP1.1 (A), U2.1 (IN), U2.3 (EN)
- net +1V8: now reaches R3.1
- net +1V8: now also C4.1, R1.1, U1.4 (VDD), JP1.3 (B), TP2.1, U2.5 (OUT)
- removed net VDD: C4.1, R1.1, R2.1, U1.4 (VDD), U1.5 (VDDIO)
- new net: R3.2, R4.1, U2.4 (FB)
- new net VCC: JP1.2 (C), R2.1, TP1.1, U1.5 (VDDIO)
- no-connect marks 5 -> 0
Other:
- note removed: "VDD: 1.8~2.1V"
- moved on the sheet: C1, C2, C3, C4, R1, R2, U1
