File: pmw3360_pcb_pinheader/pmw3360_pcb_pinheader.kicad_sch (KiCad schematic)
At the start: 15 parts, among them J1 Conn_01x08, U1 PMW3360DM-T2QU, U2 TPS73601DBV

Commit message: Update rev2.2
Parts:
- added H1, H2, H3, H4: MountingHole_Pad, MountingHole:MountingHole_3.2mm_M3_ISO14580, symbol Mechanical:MountingHole
- added R5: 56.2k, Resistor_SMD:R_0603_1608Metric_Pad0.98x0.95mm_HandSolder, symbol Device:R
- JP1: footprint Jumper:SolderJumper-3_P1.3mm_Open_Pad1.0x1.5mm_NumberLabels -> Jumper:SolderJumper-3_P1.3mm_Open_RoundedPad1.0x1.5mm_NumberLabels
- R1: value 39R -> 10k; now not fitted
- R3: value Adj_R1 -> 39R
- R4: value Adj_R2 -> 28k
- TP1: value VIO TestPoint -> VIO
- TP2: value VDD TestPoint -> VDD
- TP3: value GND TestPoint -> GND
Connections:
- net CS: now also J1.3 (Pin_3); no longer J1.5 (Pin_5)
- net GND: now also J1.1 (Pin_1), R5.2; no longer J1.8 (Pin_8), R4.2
- net MOSI: now also J1.5 (Pin_5); no longer J1.3 (Pin_3)
- net MOTION: now also J1.7 (Pin_7); no longer J1.1 (Pin_1)
- net RESET: now also J1.8 (Pin_8), R1.2; no longer J1.6 (Pin_6)
- net SCLK: now also J1.6 (Pin_6); no longer J1.2 (Pin_2)
- net VDD: now also R4.1; no longer R1.1
- net at U1.15 (LED_P): now also R3.2; no longer R1.2
- net V_IN renamed V_{IN}
- net V_{IN}: now also J1.2 (Pin_2); no longer J1.7 (Pin_7)
- net V_IO renamed V_{IO}
- net V_{IO}: now also R1.1
- new net: R4.2, R5.1, U2.4 (FB)
Other:
- note added: "LDO can be replace by RT9193-18GB: - Change C3 and C4 to 1uF. - Change R5 to a 22nF or larger ceramic capacitor. - R4 don't install."
- note added: "Mounting Holes"
- note added: "Operating Voltage Range VIN: 2.0~5.5V, must be same or greater than V_{DD} + 0.2V VDD: 1.8~2.1V, Typ. 1.9V VIO: 1.8~3.6V, Typ. 1.9V, must be same or greater than V_{DD}"
- note added: "Reserved, ~{RESET} pin has a built in weak pull up circuit."
- note added: "Test Points"
- note removed: "V_{DD} = (Adj_R1 + Adj_R2)/Adj_R2 * 1.204 Adj_R1 || Adj_R2 ~= 19k ohm V_{DD} Adj_R1 Adj_R2 1.8V 28k 56.2k 2.5V 39.2k 36.5k"
- note removed: "V_{IN}: 2.0~5.5V, must be same or greater than V_{DD} + 0.2V V_{DD}: 1.8~2.1V, Typ. 1.9V V_{IO}: 1.8~3.6V, Typ. 1.9V, must be same or greater than V_{DD}"
- moved on the sheet: TP1, TP2, TP3
