File: pmw3360_pcb_pinheader/pmw3360_pcb_pinheader.kicad_pcb (KiCad board)
At the start: 2 copper layers, 26.2 x 35.1 mm, 19 parts, among them J1 Conn_01x08, U1 PMW3360DM-T2QU, U2 TPS73601DBV

Commit message: Update rev2.2
Parts:
- removed REF** (x4): MountingHole_3.2mm_M3_DIN965_Pad, MountingHole:MountingHole_3.2mm_M3_DIN965_Pad
- added H1: MountingHole_Pad, MountingHole:MountingHole_3.2mm_M3_ISO14580, F.Cu at (136.9, 79.5)
- added H2: MountingHole_Pad, MountingHole:MountingHole_3.2mm_M3_ISO14580, F.Cu at (136.9, 106.5)
- added H3: MountingHole_Pad, MountingHole:MountingHole_3.2mm_M3_ISO14580, F.Cu at (154.4, 79.5)
- added H4: MountingHole_Pad, MountingHole:MountingHole_3.2mm_M3_ISO14580, F.Cu at (154.4, 106.5)
- added R1: 10k, Resistor_SMD:R_0603_1608Metric_Pad0.98x0.95mm_HandSolder, F.Cu at (154.1, 85.3)
- JP1: footprint Jumper:SolderJumper-3_P1.3mm_Open_Pad1.0x1.5mm_NumberLabels -> Jumper:SolderJumper-3_P1.3mm_Open_RoundedPad1.0x1.5mm_NumberLabels
- R4: renamed from R3; value Adj_R1 -> 28k
- R5: renamed from R4; value Adj_R2 -> 56.2k
- TP1: value VDDIO TestPoint -> VIO TestPoint
- moved TP1 101.9 mm to (145.6, 80.0)
- moved JP1 101.5 mm to (153.9, 90.3)
- moved R3 100.3 mm to (143.9, 103.3)
- moved C1 100.3 mm to (154.1, 94.3)
- moved C2 100.3 mm to (154.1, 96.0)
- moved U1 100.1 mm to (145.6, 92.5)
- moved R4 100.0 mm to (149.7, 106.3)
- moved R5 100.0 mm to (149.7, 108.0)
- moved C3 100.0 mm to (140.9, 107.1)
- moved C4 100.0 mm to (147.1, 107.1)
- moved U2 100.0 mm to (144.1, 107.1)
- moved TP3 98.8 mm to (142.4, 80.0)
- moved TP2 95.9 mm to (148.9, 80.0)
- moved J1 92.9 mm to (135.4, 101.9), turned to 180 degrees
- moved R2 91.7 mm to (154.1, 83.5)
- renumbered R1 to R3
Connections:
- net V_IO renamed V_{IO}
- C3 pad 1: V_IN -> V_{IN}
- J1 pad 1: /MOTION -> GND
- J1 pad 2: /SCLK -> V_{IN}
- J1 pad 3: /MOSI -> /CS
- J1 pad 5: /CS -> /MOSI
- J1 pad 6: /RESET -> /SCLK
- J1 pad 7: V_IN -> /MOTION
- J1 pad 8: GND -> /RESET
- JP1 pad 1: V_IN -> V_{IN}
- U2 pad 1: V_IN -> V_{IN}
- U2 pad 3: V_IN -> V_{IN}
Routing:
- net GND: track 142.7 -> 15.1 mm, vias 15 -> 9
- net V_IN: track 51.9 -> 0.00 mm, vias 2 -> 0
- net V_{IN}: track 0.00 -> 45.2 mm, vias 0 -> 2
- net /RESET: track 36.9 -> 22.6 mm
- net VDD: track 58.5 -> 49.4 mm, vias 0 -> 2
- net V_{IO}: track 25.7 -> 22.2 mm
- net /MISO: track 27.3 -> 29.6 mm, vias 0 -> 1
- net /MOTION: track 6.55 -> 5.45 mm
- net Net-(U1-LED_P): track 11.5 -> 10.4 mm
- net Net-(U1-VDDPIX): track 6.17 -> 5.30 mm
Other:
- board size 26.2 x 35.1 mm -> 23.5 x 33 mm
- board text added: "CS"
- board text added: "MISO"
- board text added: "MOSI"
- board text added: "Reset"
- board text added: "SCLK"
- board text removed: "SCK"
- board text removed: "SI"
- board text removed: "SO"
- board text removed: "~{CS}"
- board text removed: "~{RST}"

Commit message: Update silkscreen text
Other:
- board text added: "${TITLE} Rev ${REVISION}"
- board text removed: "PMW3360 PCB Rev 2.1"
Changed lines of the file:
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@@
     (effects (font (size 1 1) (thickness 0.15)) (justify left mirror))
   )
-  (gr_text "PMW3360 PCB\nRev 2.1" (at 149.939 79.2338) (layer "B.SilkS")
+  (gr_text "${TITLE}\nRev ${REVISION}" (at 149.939 79.2338) (layer "B.SilkS")
     (effects (font (size 1 1) (thickness 0.15)) (justify left top mirror))
   )
