File: pmw3360_pcb_ffc/pmw3360_pcb_ffc.kicad_pcb (KiCad board)
At the start: 2 copper layers, 27 x 22.5 mm, 20 parts, among them J1 Interface, U1 PMW3360DM-T2QU, U2 TPS73601DBV

Commit message: Update designators
Parts:
- removed R5: 56.2k, Resistor_SMD:R_0603_1608Metric_Pad0.98x0.95mm_HandSolder
- added C5: 22nF, Capacitor_SMD:C_0603_1608Metric_Pad1.08x0.95mm_HandSolder, F.Cu at (160.5, 88.7)
- C4: value 4.7uF -> 1uF
- U1: value PMW3360DM-T2QU -> PMW3360
- U2: value TPS73601DBV -> TLV74318PDBVR
- moved TP2 0.27 mm to (158.7, 97.2)
- moved TP3 0.22 mm to (161.0, 97.3)
Routing:
- net Net-(U1-VDDPIX): track 5.86 -> 4.11 mm
- net GND: track 107.2 -> 107.3 mm, vias 7 -> 8
