File: pmw3360_pcb_ffc/pmw3360_pcb_ffc.kicad_sch (KiCad schematic)
At the start: 20 parts, among them J1 Interface, U1 PMW3360DM-T2QU, U2 TPS73601DBV

Commit message: Update designators
Parts:
- removed R5: 56.2k, Resistor_SMD:R_0603_1608Metric_Pad0.98x0.95mm_HandSolder, symbol Device:R
- removed U2: TPS73601DBV, Package_TO_SOT_SMD:SOT-23-5, symbol Regulator_Linear:TPS73601DBV
- added C5: 22nF, Capacitor_SMD:C_0603_1608Metric_Pad1.08x0.95mm_HandSolder, symbol Device:C_Small
- added U2: TLV74318PDBVR, Package_TO_SOT_SMD:SOT-23-5, symbol PMW3360_PCB:TLV74318PDBVR
- C4: value 4.7uF -> 1uF
- R4: now not fitted
- U1: value PMW3360DM-T2QU -> PMW3360
Connections:
- net GND: now also C5.2, U2.2 (GND)
- net VDD: now also U2.5 (OUT)
- net V_{IN}: now also U2.1 (IN), U2.3 (EN)
- net at R4.2: now also C5.1, U2.4 (NC)
Other:
- note added: "LDO selection: a) TLV74318PDBVR (Fixed 1.8V output): * C3 and C4: 1uF * C5 and R4: don't install b) RT9193-18GB (Fixed 1.8V output): * C3 and C4: 1uF * C5: 22nF or larger ceramic capacitor * R4: don't install c) TPS73601DBV: * C3: 1uF * C4: 4.7uF * C5: 56.2kΩ * R4: 28kΩ"
- note added: "Operating voltage range: * VIN: Depends on config * VIO: VDD ~ 3.6V * VDD: 1.8 ~ 2.1V"
- note added: "Voltage-Level config: a) 3.3V: * VIN: connect to 3.3V, 3.6V max * JP1: [1-2 3], VIO=VIN b) 1.8V with LDO: * VIN: (VDD + 0.2V) ~ 5.5V * JP1: [1 2-3], VIO=VDD c) 1.8V without LDO: * VIN: connect to 1.8V, 2.1V max * JP1: [1-2-3], VIO=VDD=VIN * U2, R4, C3~5 can be omitted as well"
- note removed: "LDO can be replace by RT9193-18GB: - Change C3 and C4 to 1uF. - Change R5 to a 22nF or larger ceramic capacitor. - R4 don't install."
- note removed: "Operating Voltage Range VIN: 2.0~5.5V, must be same or greater than V_{DD} + 0.2V VDD: 1.8~2.1V, Typ. 1.9V VIO: 1.8~3.6V, Typ. 1.9V, must be same or greater than V_{DD}"
- moved on the sheet: C1, C2, C3, C4, J1, JP1, R1, R2, R3, TP1, TP2, TP3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
