File: pmw3360_pcb_jst/pmw3360_pcb_jst.kicad_pcb (KiCad board)
At the start: 2 copper layers, 27 x 28 mm, 20 parts, among them J1 Conn_01x08, U1 PMW3360DM-T2QU, U2 TPS73601DBV

Commit message: Update designators
Parts:
- removed R5: 56.2k, Resistor_SMD:R_0603_1608Metric_Pad0.98x0.95mm_HandSolder
- added C5: 22nF, Capacitor_SMD:C_0603_1608Metric_Pad1.08x0.95mm_HandSolder, F.Cu at (190.8, 140.9)
- JP1: footprint Jumper:SolderJumper-3_P1.3mm_Open_Pad1.0x1.5mm_NumberLabels -> Jumper:SolderJumper-3_P1.3mm_Open_RoundedPad1.0x1.5mm_NumberLabels
- TP1, TP2, TP3: footprint TestPoint:TestPoint_Pad_D1.5mm -> TestPoint:TestPoint_Pad_D1.0mm
- U2: value TPS73601DBV -> TLV74318PDBVR
